File: xorne-pcb/xorne-pcb.kicad_pcb (KiCad board)
At the start: 2 copper layers, 133.8 x 92.2 mm, 56 parts, among them SW1 SW_PUSH, SW10 SW_PUSH, SW11 SW_PUSH, SW12 SW_PUSH, SW13 SW_PUSH, SW14 SW_PUSH, SW15 SW_PUSH, SW16 SW_PUSH, SW17 SW_PUSH, SW18 SW_PUSH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

Commit message: save pin changes
Routing:
- net Net-(D19-Pad2): track 75.6 -> 72.9 mm, vias 2 -> 1
- net Net-(D12-Pad2): track 22.3 -> 23.9 mm, vias 0 -> 1
- net Net-(D18-Pad2): track 40.9 -> 42.5 mm, vias 0 -> 1
- net Net-(D17-Pad2): track 63.1 -> 64.5 mm, vias 0 -> 1
- net Net-(D16-Pad2): track 88.9 -> 90.3 mm, vias 0 -> 1
- net col3: track 197.5 -> 196.1 mm
